File: hardware/ese-rust-board/LED_STRIP.kicad_sch (KiCad schematic)
At the start: 20 parts

Commit message: align symbols, footprints and MPNs/GPNs
Parts:
- D401, D402, D403, D404, D405, D406, D407, D408, D409, D410: footprint (none) -> LED_SMD:LED_0603_1608Metric; MPN (none) -> 150060BS75000
- R401, R402, R403, R404, R405, R406, R407, R408, R409, R410: value 470R -> 330R; footprint (none) -> Resistor_SMD:R_0603_1608Metric; MPN (none) -> GPR0603330R

Commit message: fix: LED strip to +5V, R to 1k, add note about active low
Parts:
- R401, R402, R403, R404, R405, R406, R407, R408, R409, R410: value 330R -> 1k; MPN GPR0603330R -> GPR06031K
Connections:
- net +3V3 renamed +5V
Other:
- note added: "Note: LEDs are active low, the GPIOs have to be set to LOW for the LED to be on."
Changed lines of the file:
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@@
 		(company "Systemscape GmbH")
+	)
+	(text "Note: LEDs are active low,\nthe GPIOs have to be set to\nLOW for the LED to be on."
+		(exclude_from_sim no)
+		(at 70.104 28.194 0)
+		(effects
+			(font
+				(size 1.27 1.27)
+				(thickness 0.1588)
+			)
+			(justify left)
+		)
 	)
 	(junction
@@
 			)
 			(justify left)
+		)
+	)
+	(symbol
+		(lib_id "power:+5V")
+		(at 25.4 22.86 0)
+		(unit 1)
+		(body_style 1)
+		(exclude_from_sim no)
+		(in_bom yes)
+		(on_board yes)
+		(in_pos_files yes)
+		(dnp no)
+		(fields_autoplaced yes)
+		(property "Reference" "#PWR0401"
+			(at 25.4 26.67 0)
+			(hide yes)
+			(show_name no)
+			(do_not_autoplace no)
+			(effects
+				(font
+					(size 1.27 1.27)
+				)
+			)
+		)
+		(property "Value" "+5V"
+			(at 25.4 17.78 0)
+			(show_name no)
+			(do_not_autoplace no)
+			(effects
+				(font
+					(size 1.27 1.27)
+				)
+			)
+		)
+		(property "Footprint" "Package_LCC:PLCC-84_29.3x29.3mm_P1.27mm"
+			(at 25.4 22.86 0)
+			(hide yes)
+			(show_name no)
+			(do_not_autoplace no)
+			(effects
+				(font
+					(size 1.27 1.27)
+				)
+			)
+		)
+		(property "Datasheet" ""
+			(at 25.4 22.86 0)
+			(hide yes)
+			(show_name no)
+			(do_not_autoplace no)
+			(effects
+				(font
+					(size 1.27 1.27)
+				)
+			)
+		)
+		(property "Description" "Power symbol creates a global label with name \"+5V\""
+			(at 25.4 22.86 0)
+			(hide yes)
+			(show_name no)
+			(do_not_autoplace no)
+			(effects
+				(font
+					(size 1.27 1.27)
+				)
+			)
+		)
+		(pin "1"
+		)
+		(instances
+			(project "ese-rust-board"
+				(path "/66810f2f-e65f-4576-8743-4cd701ccca60/9da36eb9-c061-4a6c-ab15-3acd5db13b6c"
+					(reference "#PWR0401")
+					(unit 1)
+				)
+			)
 		)
 	)
@@
 			)
 		)
-		(property "Value" "330R"
+		(property "Value" "1k"
 			(at 33.02 77.47 90)
 			(show_name no)
@@
 			)
 		)
-		(property "MPN" "GPR0603330R"
+		(property "MPN" "GPR06031K"
 			(at 33.02 80.01 90)
 			(hide yes)
@@
 			)
 		)
-		(property "Value" "330R"
+		(property "Value" "1k"
 			(at 33.02 68.58 90)
 			(show_name no)
@@
 			)
 		)
-		(property "MPN" "GPR0603330R"
+		(property "MPN" "GPR06031K"
 			(at 33.02 71.12 90)
 			(hide yes)
@@
 			)
 		)
-		(property "Value" "330R"
+		(property "Value" "1k"
 			(at 33.02 50.8 90)
 			(show_name no)
@@
 			)
 		)
-		(property "MPN" "GPR0603330R"
+		(property "MPN" "GPR06031K"
 			(at 33.02 53.34 90)
 			(hide yes)
@@
 			)
 		)
-		(property "Value" "330R"
+		(property "Value" "1k"
 			(at 33.02 86.36 90)
 			(show_name no)
@@
 			)
 		)
-		(property "MPN" "GPR0603330R"
+		(property "MPN" "GPR06031K"
 			(at 33.02 88.9 90)
 			(hide yes)
@@
 			)
 		)
-		(property "Value" "330R"
+		(property "Value" "1k"
 			(at 33.02 24.13 90)
 			(show_name no)
@@
 			)
 		)
-		(property "MPN" "GPR0603330R"
+		(property "MPN" "GPR06031K"
 			(at 33.02 26.67 90)
 			(hide yes)
@@
 			)
 		)
-		(property "Value" "330R"
+		(property "Value" "1k"
 			(at 33.02 41.91 90)
 			(show_name no)
@@
 			)
 		)
-		(property "MPN" "GPR0603330R"
+		(property "MPN" "GPR06031K"
 			(at 33.02 44.45 90)
 			(hide yes)
@@
 				(path "/66810f2f-e65f-4576-8743-4cd701ccca60/9da36eb9-c061-4a6c-ab15-3acd5db13b6c"
 					(reference "R403")
-					(unit 1)
-				)
-			)
-		)
-	)
-	(symbol
-		(lib_id "power:+3V3")
-		(at 25.4 22.86 0)
-		(unit 1)
-		(body_style 1)
-		(exclude_from_sim no)
-		(in_bom yes)
-		(on_board yes)
-		(in_pos_files yes)
-		(dnp no)
-		(fields_autoplaced yes)
-		(property "Reference" "#PWR0401"
-			(at 25.4 26.67 0)
-			(hide yes)
-			(show_name no)
-			(do_not_autoplace no)
-			(effects
-				(font
-					(size 1.27 1.27)
-				)
-			)
-		)
-		(property "Value" "+3V3"
-			(at 25.4 17.78 0)
-			(show_name no)
-			(do_not_autoplace no)
-			(effects
-				(font
-					(size 1.27 1.27)
-				)
-			)
-		)
-		(property "Footprint" "Package_DFN_QFN:Diodes_UDFN3810-9_TYPE_B"
-			(at 25.4 22.86 0)
-			(hide yes)
-			(show_name no)
-			(do_not_autoplace no)
-			(effects
-				(font
-					(size 1.27 1.27)
-				)
-			)
-		)
-		(property "Datasheet" ""
-			(at 25.4 22.86 0)
-			(hide yes)
-			(show_name no)
-			(do_not_autoplace no)
-			(effects
-				(font
-					(size 1.27 1.27)
-				)
-			)
-		)
-		(property "Description" "Power symbol creates a global label with name \"+3V3\""
-			(at 25.4 22.86 0)
-			(hide yes)
-			(show_name no)
-			(do_not_autoplace no)
-			(effects
-				(font
-					(size 1.27 1.27)
-				)
-			)
-		)
-		(pin "1"
-		)
-		(instances
-			(project "ese-rust-board"
-				(path "/66810f2f-e65f-4576-8743-4cd701ccca60/9da36eb9-c061-4a6c-ab15-3acd5db13b6c"
-					(reference "#PWR0401")
 					(unit 1)
 				)
@@
 			)
 		)
-		(property "Value" "330R"
+		(property "Value" "1k"
 			(at 33.02 104.14 90)
 			(show_name no)
@@
 			)
 		)
-		(property "MPN" "GPR0603330R"
+		(property "MPN" "GPR06031K"
 			(at 33.02 106.68 90)
 			(hide yes)
@@
 			)
 		)
-		(property "Value" "330R"
+		(property "Value" "1k"
 			(at 33.02 59.69 90)
 			(show_name no)
@@
 			)
 		)
-		(property "MPN" "GPR0603330R"
+		(property "MPN" "GPR06031K"
 			(at 33.02 62.23 90)
 			(hide yes)
@@
 			)
 		)
-		(property "Value" "330R"
+		(property "Value" "1k"
 			(at 33.02 95.25 90)
 			(show_name no)
@@
 			)
 		)
-		(property "MPN" "GPR0603330R"
+		(property "MPN" "GPR06031K"
 			(at 33.02 97.79 90)
 			(hide yes)
@@
 			)
 		)
-		(property "Value" "330R"
+		(property "Value" "1k"
 			(at 33.02 33.02 90)
 			(show_name no)
@@
 			)
 		)
-		(property "MPN" "GPR0603330R"
+		(property "MPN" "GPR06031K"
 			(at 33.02 35.56 90)
 			(hide yes)

Commit message: chore: work on routing a bit
Connections:
- net LED_STRIP_1: now also D410.1 (K); no longer D401.1 (K)
- net LED_STRIP_10: now also D401.1 (K); no longer D410.1 (K)
- net LED_STRIP_2: now also D409.1 (K); no longer D402.1 (K)
- net LED_STRIP_3: now also D408.1 (K); no longer D403.1 (K)
- net LED_STRIP_4: now also D407.1 (K); no longer D404.1 (K)
- net LED_STRIP_5: now also D406.1 (K); no longer D405.1 (K)
- net LED_STRIP_6: now also D405.1 (K); no longer D406.1 (K)
- net LED_STRIP_7: now also D404.1 (K); no longer D407.1 (K)
- net LED_STRIP_8: now also D403.1 (K); no longer D408.1 (K)
- net LED_STRIP_9: now also D402.1 (K); no longer D409.1 (K)
